File: hw/R2P_IMU_module.brd (EAGLE design)
At the start: 40 x 40 mm, 32 parts, among them U1 STM32F103CX, U5 LD3985XX, X1 MICROMATCH-4

Commit message: Ongoing layout
Parts:
- added C10: 470n, rcl:C0603
- added C13: 10n, rcl:C0603
- added C14: 220n, rcl:C0603
- added C15: 4.7u, rcl:C0805
- added C16, C2, C4: 10u, rcl:C0805
- added C17, C3, C8: 100n, rcl:C0603
- added R5: 10k, rcl:R0603
- added R6, R7: 2.7k, rcl:R0603
- added U$2: LPS331AP, st:HCLGA16
- added U2: L3G4200D, st:LGA16
- added U6: LSM303DLHC, st:LGA14
- added X2: MICROMATCH-6, tyco:MICROMATCH-6
- X1: device con-amp-micromatch:MICROMATCH-4 -> tyco:MICROMATCH-4
- moved X1 0.63 mm to (34.3, 37.1)
Connections:
- new net BAR_CS: U$2.P$8
- new net BAR_INT1: U$2.P$11
- new net BAR_INT2: U$2.P$9
- new net N$10: C10.1, C13.1, U2.P$14
- new net N$14: C14.1, U6.12
- new net N$16: C14.2, U6.13
- new net N$17: C15.1, U6.6
- new net N$9: C10.2, R5.1
- net +3V3: now also C16.1, C17.1, C2.1, C3.1, C4.1, C8.1, R6.1, R7.1, U$2.P$1, U$2.P$14, U$2.P$15, U2.P$1, U2.P$15, U2.P$16, U6.1, U6.14, X2.3
- net AM_DRDY: now also U6.9
- net AM_INT1: now also U6.5
- net AM_INT2: now also U6.4
- net GND: now also C13.2, C15.2, C16.2, C17.2, C2.2, C3.2, C4.2, C8.2, R5.2, U$2.P$10, U$2.P$12, U$2.P$13, U$2.P$16, U$2.P$5, U2.P$10, U2.P$11, U2.P$12, U2.P$13, U2.P$8, U2.P$9, U6.10, U6.11, U6.7, X2.1
- net GPS_RESET: now also X2.5
- net GPS_RX: now also X2.2
- net GPS_STATUS: now also X2.6
- net GPS_TX: now also X2.4
- net GYRO_CS: now also U2.P$5
- net GYRO_INT1: now also U2.P$7
- net GYRO_INT2: now also U2.P$6
- net MISO: now also U$2.P$7, U2.P$4
- net MOSI: now also U$2.P$6, U2.P$3
- net SCK: now also U$2.P$4, U2.P$2
- net SCL: now also R7.2, U6.2
- net SDA: now also R6.2, U6.3
Routing:
- net GPS_RESET: track 0.00 -> 26.4 mm, vias 0 -> 1
- net SDA: track 0.00 -> 24.4 mm, vias 0 -> 2
- net GPS_RX: track 0.00 -> 22.7 mm, vias 0 -> 1
- net SCL: track 0.00 -> 22.5 mm, vias 0 -> 2
- net AM_INT1: track 0.00 -> 20.5 mm, vias 0 -> 2
- net AM_INT2: track 0.00 -> 20.3 mm, vias 0 -> 2
- net SCK: track 0.00 -> 16.8 mm, vias 0 -> 3
- net MOSI: track 0.00 -> 14.8 mm, vias 0 -> 2
- net AM_DRDY: track 0.00 -> 14.6 mm, vias 0 -> 2
- net +3V3: track 112.4 -> 126.8 mm
- net MISO: track 0.00 -> 13.2 mm, vias 0 -> 2
- net GYRO_INT1: track 0.00 -> 12.4 mm
- net N$10: track 0.00 -> 3.91 mm
- net GYRO_CS: track 0.00 -> 3.02 mm, vias 0 -> 2
- net N$14: track 0.00 -> 2.07 mm
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
Commit message: Board layout finished
Parts:
- moved C11 12.1 mm to (26.0, 36.4), turned to 90 degrees
- moved R3 10.9 mm to (28.1, 36.4), turned to 270 degrees
- moved U$1 7.33 mm to (27.0, 33.0), turned to 180 degrees
- moved X1 1.91 mm to (34.3, 35.2)
- moved X2 1.91 mm to (6.99, 35.2)
- moved C13 1.35 mm to (9.84, 29.2)
- moved R5 1.35 mm to (9.84, 31.3)
- moved C10 1.06 mm to (12.4, 30.6)
- moved C8 0.32 mm to (21.6, 36.8)
- moved C2 0.16 mm to (23.7, 36.8)
Connections:
- removed net N$1: U$4.P$5
- removed net OSC_OUT: U1.6
- net +3V3: now also X2.1; no longer X2.3
- net BAR_CS: now also U1.4
- net BAR_INT1: now also U1.2
- net BAR_INT2: now also U1.3
- net GND: now also U$4.P$5, X2.2; no longer X2.1
- net GPS_RX: now also X2.4; no longer X2.2
- net GPS_TX: now also X2.3; no longer X2.4
Routing:
- net +3V3: track 126.8 -> 198.1 mm, vias 11 -> 14
- net GPS_STATUS: track 0.00 -> 24.0 mm
- net GPS_TX: track 0.00 -> 21.6 mm, vias 0 -> 1
- net BAR_INT1: track 0.00 -> 14.4 mm, vias 0 -> 2
- net BAR_INT2: track 0.00 -> 13.0 mm, vias 0 -> 2
- net BAR_CS: track 0.00 -> 12.9 mm, vias 0 -> 2
- net GYRO_INT2: track 0.00 -> 11.4 mm, vias 0 -> 2
- net GYRO_CS: track 3.02 -> 9.79 mm
- net OSC_IN: track 11.2 -> 5.30 mm
- net N$17: track 0.00 -> 2.27 mm
- net GPS_RX: track 22.7 -> 24.7 mm
- net UART_RX: track 38.7 -> 36.8 mm
- net UART_TX: track 43.2 -> 41.2 mm
- net +5V: track 53.3 -> 51.4 mm
- net GYRO_INT1: track 12.4 -> 13.5 mm
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